File: kicad/tinyispmicro.sch (KiCad schematic (older format))
At the start: 16 parts, among them J1 AVRISP6, P1 PGM, P2 REG, P3 MODE, P4 USB, U1 10p, U2 150, U3 MCP1824, U4 ATTINYX4, U5 1u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

Commit message: fix part number for USB connector
Parts:
- P4: Digikey 151-1206-1-ND -> H11671CT-ND
Changed lines of the file:
@@
 LIBS:zener-sot23-3
 LIBS:network0606
+LIBS:tinyispmicro-cache
 EELAYER 27 0
 EELAYER END
@@
 Sheet 1 1
 Title ""
-Date "13 nov 2014"
+Date "18 dec 2014"
 Rev ""
 Comp ""
@@
 F 2 "USB-MiniB" H 8200 2650 60  0000 C CNN
 F 3 "NOTE: Break off plastic grabbers." H 8150 2050 60  0000 C CNN
-F 4 "151-1206-1-ND" V 8200 2650 60  0001 C CNN "Digikey"
+F 4 "H11671CT-ND" V 8200 2650 60  0001 C CNN "Digikey"
 F 5 ".41" V 8200 2650 60  0001 C CNN "Cost1"
 	1    8200 2650

Commit message: fix price
Parts:
- P4: Cost1 .41 -> .80
Changed lines of the file:
@@
 F 3 "NOTE: Break off plastic grabbers." H 8150 2050 60  0000 C CNN
 F 4 "H11671CT-ND" V 8200 2650 60  0001 C CNN "Digikey"
-F 5 ".41" V 8200 2650 60  0001 C CNN "Cost1"
+F 5 ".80" V 8200 2650 60  0001 C CNN "Cost1"
 	1    8200 2650
 	1    0    0    -1
