File: kicad/tinyispmicro.kicad_pcb (KiCad board)
At the start: 2 copper layers, 36.8 x 16.5 mm, 16 parts, among them J1 AVRISP6, P1 PGM, P2 REG, P3 MODE, P4 USB, U3 MCP1824, U4 ATTINYX4, U6 1.5k, U7 33, X1 12MHz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

Commit message: add new rev and update design
Routing:
- net (no net): track 0.00 -> 13.0 mm
- net +5V: track 70.2 -> 75.1 mm, vias 0 -> 3
- net GND: track 76.9 -> 81.0 mm, vias 4 -> 8
- net N-0000013: track 15.1 -> 13.2 mm, vias 2 -> 0
Other:
- net class Default: via_drill 0.635 -> 0.508
- board text added: "(C) 2017 C. Lohr"
- board text added: "REV A"
- board text added: "http://github.com/cnlohr/tinyisp-micro"
- board text removed: "(C) 2014 C. Lohr"
- board text removed: "REV -"
